File: batteryNode/PCB/batteryNode.sch (KiCad schematic (older format))
At the start: 55 parts, among them J100 cell_taps, J101 therm_conn, J200 ISP_Header, J300 Conn_01x06, Q100 IRLML9303TRPBF, SW200 SW_Push, U100 BQ76925RGER, U200 ATtiny2313A-MU, U300 LTC2875-DD, Y200 10MHz

Commit message: added current control. Started V2 of layout
Parts:
- added Q101: NMOS, Package_SO:PowerPAK_SO-8_Single, symbol Device:Q_NMOS_DGS
- added R209: 10k, Resistor_SMD:R_0603_1608Metric, symbol Device:R
- added U101: MIC5060, Package_DFN_QFN:MLF-8-1EP_3x3mm_P0.65mm_EP1.55x2.3mm, symbol batteryNodeLib:MIC5060
- J101: value therm_conn -> load
Connections:
- net GND: now also J101.2 (Pin_2), Q101.1 (S), R209.2, U101.3 (SOURCE), U101.4 (GND)
- net tap6: now also U101.1 (V+)
- net v_iout: now reaches U100.14 (VIOUT)
- net v_iout: now also R207.2
- net i_ctrl: now reaches U200.7 (PD5)
- net i_ctrl: now also R209.1, U101.2 (INPUT)
- net therm_in: no longer names the net of J101.1 (Pin_1)
- net therm_in: now also Q101.8 (D); no longer R207.2
- net therm_in_filt renamed v_iout_filt
- net therm_out: no longer names the net of U100.16 (VTB)
- net therm_out: no longer J101.2 (Pin_2)
- new net: Q101.4 (G), U101.5 (GATE)
- no-connect marks 11 -> 14
Other:
- note added: "Low Side Current Control\n"
- moved on the sheet: C101, C102, C103, C104, C105, C106, C107, C108, C109, C300, D10, FB300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

Commit message: Old changes made that I can't remember
Hopefully I don't have to roll the project back :)
Connections:
- net MISO_SDA is gone; now on net MISO: J200.1 (Pin_1)
- net MOSI is gone; now on net MOSI_SDA: J200.4 (Pin_4)
- net at C202.1, R204.1, Y200.2: now also U200.3 (PA0/XTAL1); no longer U200.2 (PA1/XTAL2)
- net at C201.1, R204.2, Y200.1: now also U200.2 (PA1/XTAL2); no longer U200.3 (PA0/XTAL1)
Changed lines of the file:
@@
 	1    0    0    -1
 $EndComp
-Wire Wire Line
-	10650 5850 10950 5850
-Wire Wire Line
-	10650 5750 10950 5750
-Wire Wire Line
-	10950 5750 10950 5600
-Wire Wire Line
-	10650 5950 10950 5950
-Wire Wire Line
-	10950 5950 10950 6100
 $Comp
 L power:GND #PWR0101
 U 1 1 5D0D893C
-P 10950 6100
-F 0 "#PWR0101" H 10950 5850 50  0001 C CNN
-F 1 "GND" H 10955 5927 50  0000 C CNN
-F 2 "" H 10950 6100 50  0001 C CNN
-F 3 "" H 10950 6100 50  0001 C CNN
-	1    10950 6100
+P 11000 6100
+F 0 "#PWR0101" H 11000 5850 50  0001 C CNN
+F 1 "GND" H 11005 5927 50  0000 C CNN
+F 2 "" H 11000 6100 50  0001 C CNN
+F 3 "" H 11000 6100 50  0001 C CNN
+	1    11000 6100
 	1    0    0    -1
 $EndComp
 Text Label 9700 5750 0    50   ~ 0
-MISO_SDA
+MISO
 Text Label 9700 5850 0    50   ~ 0
 SCK_SCL
 Text Label 9700 5950 0    50   ~ 0
 ~reset
-Text Label 10950 5850 2    50   ~ 0
-MOSI
+Text Label 11000 5850 2    50   ~ 0
+MOSI_SDA
 Text Label 9750 2550 2    50   ~ 0
 SCK_SCL
@@
 	7800 3500 7800 3400
 Connection ~ 7800 3000
-Wire Wire Line
-	7200 2050 8100 2050
 Connection ~ 7200 3000
 Wire Wire Line
 	7650 3000 7800 3000
 Wire Wire Line
-	7800 2250 7800 2400
-Wire Wire Line
-	7800 2250 8100 2250
-Wire Wire Line
 	7200 2050 7200 2400
 $Comp
@@
 L power:+3V3 #PWR0106
 U 1 1 5D105C11
-P 10950 5600
-F 0 "#PWR0106" H 10950 5450 50  0001 C CNN
-F 1 "+3V3" H 10965 5773 50  0000 C CNN
-F 2 "" H 10950 5600 50  0001 C CNN
-F 3 "" H 10950 5600 50  0001 C CNN
-	1    10950 5600
+P 11000 5600
+F 0 "#PWR0106" H 11000 5450 50  0001 C CNN
+F 1 "+3V3" H 11015 5773 50  0000 C CNN
+F 2 "" H 11000 5600 50  0001 C CNN
+F 3 "" H 11000 5600 50  0001 C CNN
+	1    11000 5600
 	1    0    0    -1
 $EndComp
@@
 	4150 2700 4350 2700
 $Comp
-L power:GND #PWR?
+L power:GND #PWR0132
 U 1 1 5D2F1455
 P 2450 4900
-F 0 "#PWR?" H 2450 4650 50  0001 C CNN
+F 0 "#PWR0132" H 2450 4650 50  0001 C CNN
 F 1 "GND" H 2455 4727 50  0000 C CNN
 F 2 "" H 2450 4900 50  0001 C CNN
@@
 F 1 "NMOS" H 2556 4255 50  0000 L CNN
 F 2 "Package_SO:PowerPAK_SO-8_Single" H 2550 4400 50  0001 C CNN
-F 3 "~" H 2350 4300 50  0001 C CNN
+F 3 "SI7460DP-T1-GE3CT-ND" H 2350 4300 50  0001 C CNN
 	1    2350 4300
 	1    0    0    -1
@@
 Connection ~ 1100 4300
 $Comp
-L power:GND #PWR?
+L power:GND #PWR0133
 U 1 1 5D45B79C
 P 1100 4900
-F 0 "#PWR?" H 1100 4650 50  0001 C CNN
+F 0 "#PWR0133" H 1100 4650 50  0001 C CNN
 F 1 "GND" H 1105 4727 50  0000 C CNN
 F 2 "" H 1100 4900 50  0001 C CNN
@@
 	9300 3250 9950 3250
 $Comp
-L power:GND #PWR?
+L power:GND #PWR0137
 U 1 1 5D4EB2FD
 P 9950 3850
-F 0 "#PWR?" H 9950 3600 50  0001 C CNN
+F 0 "#PWR0137" H 9950 3600 50  0001 C CNN
 F 1 "GND" H 9955 3677 50  0000 C CNN
 F 2 "" H 9950 3850 50  0001 C CNN
@@
 Wire Wire Line
 	9950 3850 9950 3700
+Wire Wire Line
+	10650 5850 11000 5850
+Wire Wire Line
+	11000 5750 11000 5600
+Wire Wire Line
+	10650 5750 11000 5750
+Wire Wire Line
+	11000 5950 11000 6100
+Wire Wire Line
+	10650 5950 11000 5950
+Wire Wire Line
+	7800 2050 8100 2050
+Wire Wire Line
+	7800 2050 7800 2400
+Wire Wire Line
+	7200 2050 7750 2050
+Wire Wire Line
+	7750 2050 7750 2250
+Wire Wire Line
+	7750 2250 8100 2250
 $EndSCHEMATC
